File: EAGLE/NSE2020_1.sch (EAGLE design)
At the start: 46 parts, among them CN1 MICROSD, IC1 ADP3338-3.3, X1 MINI-USB-UX60A-MB-5ST

Commit message: camファイルとデザインルール等を追加
Parts:
- added GPIO: (no value), pinhead:PINHD-1X3
Connections:
- new net RX_3: GPIO.2, MCU1.PB11-RX3
- new net TX_3: GPIO.3, MCU1.PB10-TX3
- net GND: now also GPIO.1
Changed lines of the file:
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@@
 <part name="R12" library="rcl" library_urn="urn:adsk.eagle:library:334" deviceset="R-EU_" device="M2012" package3d_urn="urn:adsk.eagle:package:23561/2" value="10k"/>
 <part name="GND20" library="supply1" library_urn="urn:adsk.eagle:library:371" deviceset="GND" device=""/>
+<part name="GPIO" library="pinhead" library_urn="urn:adsk.eagle:library:325" deviceset="PINHD-1X3" device="" package3d_urn="urn:adsk.eagle:package:22458/2"/>
+<part name="GND21" library="supply1" library_urn="urn:adsk.eagle:library:371" deviceset="GND" device=""/>
 </parts>
 <sheets>
@@
 <instance part="GND20" gate="1" x="66.04" y="30.48" smashed="yes">
 <attribute name="VALUE" x="63.5" y="27.94" size="1.778" layer="96"/>
+</instance>
+<instance part="GPIO" gate="A" x="73.66" y="144.78" smashed="yes">
+<attribute name="NAME" x="67.31" y="150.495" size="1.778" layer="95"/>
+<attribute name="VALUE" x="67.31" y="137.16" size="1.778" layer="96"/>
+</instance>
+<instance part="GND21" gate="1" x="66.04" y="147.32" smashed="yes" rot="R270">
+<attribute name="VALUE" x="63.5" y="149.86" size="1.778" layer="96" rot="R270"/>
 </instance>
 </instances>
@@
 <pinref part="GND20" gate="1" pin="GND"/>
 <wire x1="66.04" y1="33.02" x2="66.04" y2="35.56" width="0.1524" layer="91"/>
+</segment>
+<segment>
+<pinref part="GPIO" gate="A" pin="1"/>
+<pinref part="GND21" gate="1" pin="GND"/>
+<wire x1="68.58" y1="147.32" x2="71.12" y2="147.32" width="0.1524" layer="91"/>
 </segment>
 </net>
@@
 </segment>
 </net>
+<net name="TX_3" class="5">
+<segment>
+<pinref part="MCU1" gate="G$1" pin="PB10-TX3"/>
+<pinref part="GPIO" gate="A" pin="3"/>
+<wire x1="63.5" y1="142.24" x2="71.12" y2="142.24" width="0.1524" layer="91"/>
+</segment>
+</net>
+<net name="RX_3" class="5">
+<segment>
+<pinref part="GPIO" gate="A" pin="2"/>
+<pinref part="MCU1" gate="G$1" pin="PB11-RX3"/>
+<wire x1="71.12" y1="144.78" x2="63.5" y2="144.78" width="0.1524" layer="91"/>
+</segment>
+</net>
